File: hardware/probe/file5C0EA928.sch (KiCad schematic (older format))
At the start: 2 parts

Commit message: I think I can simplify the amplifier a bit
Parts:
- added J2: CONN_01, 0xDBFB7:CAP_WIRE_CONNECTION, symbol SparkFun-Connectors:CONN_01
- added R34: 500k, 1206, symbol SparkFun-Resistors:RESISTOR1206
- R2: renamed from R?; value 1M -> 500k
- R3: renamed from R?; value 10k -> 1k
Connections:
- net labels removed: INPUT
Changed lines of the file:
@@
 EESchema Schematic File Version 4
+LIBS:probe-cache
 EELAYER 26 0
 EELAYER END
 $Descr A4 11693 8268
 encoding utf-8
-Sheet 2 17
+Sheet 3 18
 Title ""
 Date ""
@@
 U 1 1 5C0EAFBF
 P 5600 3400
-F 0 "R?" V 5500 3500 45  0000 L CNN
-F 1 "1M" V 5600 3500 45  0000 L CNN
+AR Path="/5C0EA929/5C0EAFBF" Ref="R?"  Part="1"
+AR Path="/5C1436B4/5C14385B/5C0EAFBF" Ref="R2"  Part="1"
+AR Path="/5C1436B4/5C14385F/5C0EAFBF" Ref="R4"  Part="1"
+AR Path="/5C1436B4/5C143863/5C0EAFBF" Ref="R6"  Part="1"
+AR Path="/5C1436B4/5C143867/5C0EAFBF" Ref="R8"  Part="1"
+AR Path="/5C1436B4/5C14386B/5C0EAFBF" Ref="R10"  Part="1"
+AR Path="/5C1436B4/5C14386F/5C0EAFBF" Ref="R12"  Part="1"
+AR Path="/5C1436B4/5C143873/5C0EAFBF" Ref="R14"  Part="1"
+AR Path="/5C1436B4/5C143877/5C0EAFBF" Ref="R16"  Part="1"
+AR Path="/5C1436B4/5C14387B/5C0EAFBF" Ref="R18"  Part="1"
+AR Path="/5C1436B4/5C14387F/5C0EAFBF" Ref="R20"  Part="1"
+AR Path="/5C1436B4/5C143883/5C0EAFBF" Ref="R22"  Part="1"
+AR Path="/5C1436B4/5C143887/5C0EAFBF" Ref="R24"  Part="1"
+AR Path="/5C1436B4/5C14388B/5C0EAFBF" Ref="R26"  Part="1"
+AR Path="/5C1436B4/5C14388F/5C0EAFBF" Ref="R28"  Part="1"
+AR Path="/5C1436B4/5C143893/5C0EAFBF" Ref="R30"  Part="1"
+AR Path="/5C1436B4/5C143897/5C0EAFBF" Ref="R32"  Part="1"
+F 0 "R2" V 5500 3500 45  0000 L CNN
+F 1 "500k" V 5600 3500 45  0000 L CNN
 F 2 "1206" H 5600 3550 20  0001 C CNN
 F 3 "" H 5600 3400 60  0001 C CNN
@@
 	0    1    1    0
 $EndComp
-Text HLabel 5600 3200 0    50   Input ~ 0
-INPUT
 Text HLabel 5600 3600 0    50   Input ~ 0
 OUTPUT
@@
 U 1 1 5C0EB6C7
 P 5600 4000
-F 0 "#PWR?" H 5600 4000 30  0001 C CNN
+AR Path="/5C0EA929/5C0EB6C7" Ref="#PWR?"  Part="1"
+AR Path="/5C1436B4/5C14385B/5C0EB6C7" Ref="#PWR0124"  Part="1"
+AR Path="/5C1436B4/5C14385F/5C0EB6C7" Ref="#PWR0125"  Part="1"
+AR Path="/5C1436B4/5C143863/5C0EB6C7" Ref="#PWR0126"  Part="1"
+AR Path="/5C1436B4/5C143867/5C0EB6C7" Ref="#PWR0127"  Part="1"
+AR Path="/5C1436B4/5C14386B/5C0EB6C7" Ref="#PWR0128"  Part="1"
+AR Path="/5C1436B4/5C14386F/5C0EB6C7" Ref="#PWR0129"  Part="1"
+AR Path="/5C1436B4/5C143873/5C0EB6C7" Ref="#PWR0130"  Part="1"
+AR Path="/5C1436B4/5C143877/5C0EB6C7" Ref="#PWR0131"  Part="1"
+AR Path="/5C1436B4/5C14387B/5C0EB6C7" Ref="#PWR0132"  Part="1"
+AR Path="/5C1436B4/5C14387F/5C0EB6C7" Ref="#PWR0133"  Part="1"
+AR Path="/5C1436B4/5C143883/5C0EB6C7" Ref="#PWR0134"  Part="1"
+AR Path="/5C1436B4/5C143887/5C0EB6C7" Ref="#PWR0135"  Part="1"
+AR Path="/5C1436B4/5C14388B/5C0EB6C7" Ref="#PWR0136"  Part="1"
+AR Path="/5C1436B4/5C14388F/5C0EB6C7" Ref="#PWR0137"  Part="1"
+AR Path="/5C1436B4/5C143893/5C0EB6C7" Ref="#PWR0138"  Part="1"
+AR Path="/5C1436B4/5C143897/5C0EB6C7" Ref="#PWR0139"  Part="1"
+F 0 "#PWR0139" H 5600 4000 30  0001 C CNN
 F 1 "GND" H 5600 3930 30  0001 C CNN
 F 2 "" H 5600 4000 50  0001 C CNN
@@
 AR Path="/5C0EB909" Ref="R?"  Part="1"
 AR Path="/5C0EA929/5C0EB909" Ref="R?"  Part="1"
-F 0 "R?" V 5550 3900 45  0000 L CNN
-F 1 "10k" V 5650 3900 45  0000 L CNN
+AR Path="/5C1436B4/5C14385B/5C0EB909" Ref="R3"  Part="1"
+AR Path="/5C1436B4/5C14385F/5C0EB909" Ref="R5"  Part="1"
+AR Path="/5C1436B4/5C143863/5C0EB909" Ref="R7"  Part="1"
+AR Path="/5C1436B4/5C143867/5C0EB909" Ref="R9"  Part="1"
+AR Path="/5C1436B4/5C14386B/5C0EB909" Ref="R11"  Part="1"
+AR Path="/5C1436B4/5C14386F/5C0EB909" Ref="R13"  Part="1"
+AR Path="/5C1436B4/5C143873/5C0EB909" Ref="R15"  Part="1"
+AR Path="/5C1436B4/5C143877/5C0EB909" Ref="R17"  Part="1"
+AR Path="/5C1436B4/5C14387B/5C0EB909" Ref="R19"  Part="1"
+AR Path="/5C1436B4/5C14387F/5C0EB909" Ref="R21"  Part="1"
+AR Path="/5C1436B4/5C143883/5C0EB909" Ref="R23"  Part="1"
+AR Path="/5C1436B4/5C143887/5C0EB909" Ref="R25"  Part="1"
+AR Path="/5C1436B4/5C14388B/5C0EB909" Ref="R27"  Part="1"
+AR Path="/5C1436B4/5C14388F/5C0EB909" Ref="R29"  Part="1"
+AR Path="/5C1436B4/5C143893/5C0EB909" Ref="R31"  Part="1"
+AR Path="/5C1436B4/5C143897/5C0EB909" Ref="R33"  Part="1"
+F 0 "R3" V 5550 3900 45  0000 L CNN
+F 1 "1k" V 5650 3900 45  0000 L CNN
 F 2 "0603" H 5600 3950 20  0001 C CNN
 F 3 "" H 5600 3800 60  0001 C CNN
@@
 	0    1    1    0
 $EndComp
+$Comp
+L SparkFun-Resistors:RESISTOR1206 R?
+U 1 1 5C14998D
+P 5600 3000
+AR Path="/5C0EA929/5C14998D" Ref="R?"  Part="1"
+AR Path="/5C1436B4/5C14385B/5C14998D" Ref="R34"  Part="1"
+AR Path="/5C1436B4/5C14385F/5C14998D" Ref="R35"  Part="1"
+AR Path="/5C1436B4/5C143863/5C14998D" Ref="R36"  Part="1"
+AR Path="/5C1436B4/5C143867/5C14998D" Ref="R37"  Part="1"
+AR Path="/5C1436B4/5C14386B/5C14998D" Ref="R38"  Part="1"
+AR Path="/5C1436B4/5C14386F/5C14998D" Ref="R39"  Part="1"
+AR Path="/5C1436B4/5C143873/5C14998D" Ref="R40"  Part="1"
+AR Path="/5C1436B4/5C143877/5C14998D" Ref="R41"  Part="1"
+AR Path="/5C1436B4/5C14387B/5C14998D" Ref="R42"  Part="1"
+AR Path="/5C1436B4/5C14387F/5C14998D" Ref="R43"  Part="1"
+AR Path="/5C1436B4/5C143883/5C14998D" Ref="R44"  Part="1"
+AR Path="/5C1436B4/5C143887/5C14998D" Ref="R45"  Part="1"
+AR Path="/5C1436B4/5C14388B/5C14998D" Ref="R46"  Part="1"
+AR Path="/5C1436B4/5C14388F/5C14998D" Ref="R47"  Part="1"
+AR Path="/5C1436B4/5C143893/5C14998D" Ref="R48"  Part="1"
+AR Path="/5C1436B4/5C143897/5C14998D" Ref="R49"  Part="1"
+F 0 "R34" V 5500 3100 45  0000 L CNN
+F 1 "500k" V 5600 3100 45  0000 L CNN
+F 2 "1206" H 5600 3150 20  0001 C CNN
+F 3 "" H 5600 3000 60  0001 C CNN
+F 4 " " V 5684 3068 60  0000 L CNN "Field4"
+	1    5600 3000
+	0    1    1    0
+$EndComp
+$Comp
+L SparkFun-Connectors:CONN_01 J?
+U 1 1 5C14D156
+P 5700 2800
+AR Path="/5C14D156" Ref="J?"  Part="1"
+AR Path="/5C1436B4/5C14385B/5C14D156" Ref="J2"  Part="1"
+AR Path="/5C1436B4/5C14385F/5C14D156" Ref="J3"  Part="1"
+AR Path="/5C1436B4/5C143863/5C14D156" Ref="J4"  Part="1"
+AR Path="/5C1436B4/5C143867/5C14D156" Ref="J5"  Part="1"
+AR Path="/5C1436B4/5C14386B/5C14D156" Ref="J6"  Part="1"
+AR Path="/5C1436B4/5C14386F/5C14D156" Ref="J7"  Part="1"
+AR Path="/5C1436B4/5C143873/5C14D156" Ref="J8"  Part="1"
+AR Path="/5C1436B4/5C143877/5C14D156" Ref="J9"  Part="1"
+AR Path="/5C1436B4/5C14387B/5C14D156" Ref="J10"  Part="1"
+AR Path="/5C1436B4/5C14387F/5C14D156" Ref="J11"  Part="1"
+AR Path="/5C1436B4/5C143883/5C14D156" Ref="J12"  Part="1"
+AR Path="/5C1436B4/5C143887/5C14D156" Ref="J13"  Part="1"
+AR Path="/5C1436B4/5C14388B/5C14D156" Ref="J14"  Part="1"
+AR Path="/5C1436B4/5C14388F/5C14D156" Ref="J15"  Part="1"
+AR Path="/5C1436B4/5C143893/5C14D156" Ref="J16"  Part="1"
+AR Path="/5C1436B4/5C143897/5C14D156" Ref="J17"  Part="1"
+F 0 "J2" H 5657 2596 45  0000 C CNN
+F 1 "CONN_01" H 5657 2680 45  0000 C CNN
+F 2 "0xDBFB7:CAP_WIRE_CONNECTION" H 5700 3000 20  0001 C CNN
+F 3 "" H 5700 2800 50  0001 C CNN
+F 4 "" H 5657 2669 60  0000 C CNN "Field4"
+	1    5700 2800
+	-1   0    0    1
+$EndComp
 $EndSCHEMATC

Commit message: Layout complete!
Parts:
- R3: value 1k -> 10k
Changed lines of the file:
@@
 $Descr A4 11693 8268
 encoding utf-8
-Sheet 3 18
+Sheet 8 18
 Title ""
 Date ""
@@
 AR Path="/5C1436B4/5C143893/5C0EAFBF" Ref="R30"  Part="1"
 AR Path="/5C1436B4/5C143897/5C0EAFBF" Ref="R32"  Part="1"
-F 0 "R2" V 5500 3500 45  0000 L CNN
+F 0 "R32" V 5500 3500 45  0000 L CNN
 F 1 "500k" V 5600 3500 45  0000 L CNN
 F 2 "1206" H 5600 3550 20  0001 C CNN
@@
 AR Path="/5C1436B4/5C143893/5C0EB909" Ref="R31"  Part="1"
 AR Path="/5C1436B4/5C143897/5C0EB909" Ref="R33"  Part="1"
-F 0 "R3" V 5550 3900 45  0000 L CNN
-F 1 "1k" V 5650 3900 45  0000 L CNN
+F 0 "R33" V 5550 3900 45  0000 L CNN
+F 1 "10k" V 5650 3900 45  0000 L CNN
 F 2 "0603" H 5600 3950 20  0001 C CNN
 F 3 "" H 5600 3800 60  0001 C CNN
@@
 AR Path="/5C1436B4/5C143893/5C14998D" Ref="R48"  Part="1"
 AR Path="/5C1436B4/5C143897/5C14998D" Ref="R49"  Part="1"
-F 0 "R34" V 5500 3100 45  0000 L CNN
+F 0 "R49" V 5500 3100 45  0000 L CNN
 F 1 "500k" V 5600 3100 45  0000 L CNN
 F 2 "1206" H 5600 3150 20  0001 C CNN
@@
 AR Path="/5C1436B4/5C143893/5C14D156" Ref="J16"  Part="1"
 AR Path="/5C1436B4/5C143897/5C14D156" Ref="J17"  Part="1"
-F 0 "J2" H 5657 2596 45  0000 C CNN
+F 0 "J17" H 5657 2596 45  0000 C CNN
 F 1 "CONN_01" H 5657 2680 45  0000 C CNN
 F 2 "0xDBFB7:CAP_WIRE_CONNECTION" H 5700 3000 20  0001 C CNN
