File: hardware/probe/probe.kicad_pcb (KiCad board)
At the start: 2 copper layers, 87 parts, among them IC1 TLV9062IDR, IC2 AZ4580, J10 CONN_01, J11 CONN_01, J12 CONN_01, J13 CONN_01, J14 CONN_01, J15 CONN_01, J16 CONN_01, J17 CONN_01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

Commit message: Layout complete!
Parts:
- removed POWER_SUPPLY1: , 1X02
- removed R51: 1k, 0603
- removed U3: CAT24M01W, Package_SO:SOIC-8_3.9x4.9mm_P1.27mm
- added C10: 0.1uf, 0603, F.Cu at (150.8, 61.8)
- added C11: 0.1uf, 0603, F.Cu at (156.0, 75.5)
- added C6: 10uf, 0603, F.Cu at (154.1, 81.3)
- added C7: 0.1uf, 0603, F.Cu at (152.6, 78.0)
- added C8: 10UF-1206-6.3V-20%, 1206, F.Cu at (131.2, 74.0)
- added C9: 10uf, 0603, F.Cu at (137.2, 69.5)
- added J1: ISOL_3v3, 0xDBFB7:CAP_WIRE_CONNECTION, F.Cu at (161.0, 45.5)
- added J21: ISOL_3v3, 0xDBFB7:CAP_WIRE_CONNECTION, F.Cu at (163.8, 45.4)
- added J22: ISOL_3v3, 0xDBFB7:CAP_WIRE_CONNECTION, F.Cu at (166.6, 45.4)
- added J23: BATT, 0xDBFB7:CAP_WIRE_CONNECTION, F.Cu at (132.9, 77.5)
- added J24: GND, 0xDBFB7:CAP_WIRE_CONNECTION, F.Cu at (129.2, 77.6)
- added J25: GND, 0xDBFB7:CAP_WIRE_CONNECTION, B.Cu at (190.8, 42.8)
- added R54: 10k, 0603, F.Cu at (149.1, 66.7)
- added R55: 10k, 0603, F.Cu at (146.6, 67.6)
- added R56: 1k, 0603, F.Cu at (152.5, 66.7)
- added R57: 10k, 0603, F.Cu at (150.8, 65.2)
- added R58: 10k, 0603, F.Cu at (139.0, 64.9)
- added R59: 10k, 0603, F.Cu at (137.4, 75.3)
- added R60: 10k, 0603, F.Cu at (142.5, 64.9)
- added R61: 10k, 0603, F.Cu at (140.7, 75.3)
- C5: value 2.2uF -> 10uf
- IC1: footprint Package_SO:SOIC-8-1EP_3.9x4.9mm_P1.27mm_EP2.35x2.35mm -> Package_SO:SOIC-8_3.9x4.9mm_P1.27mm
- R11, R13, R15, R17, R19, R21, R23, R25, R27, R29, R3, R31, R33, R5, R7, R9: value 1k -> 10k
- R50: value 100k -> FUSE; footprint 0603 -> 1206; moved to B.Cu
- R52, R53: value 360r -> 10k
- moved R52 69.9 mm to (146.3, 74.9), turned to 180 degrees
- moved IC2 68.6 mm to (150.7, 72.0), turned to 90 degrees
- moved R53 63.4 mm to (145.4, 73.2), turned to 180 degrees
- moved U4 50.9 mm to (156.9, 79.8)
- moved U5 49.2 mm to (131.2, 68.0)
- moved J18 42.2 mm to (131.9, 49.5)
- moved C5 41.8 mm to (154.1, 78.0), turned to 270 degrees
- moved IC1 41.5 mm to (140.8, 70.1), turned to 270 degrees
- moved U1 40.9 mm to (139.9, 48.2)
- moved J19 39.8 mm to (131.9, 47.0)
- moved C4 39.2 mm to (159.9, 79.3), turned to 270 degrees
- moved J20 37.9 mm to (131.9, 52.0)
- moved R50 17.9 mm to (186.0, 42.8), turned to 0 degrees
- moved U2 13.0 mm to (149.8, 56.8), turned to 270 degrees
- moved R1 12.6 mm to (144.1, 53.9), turned to 180 degrees
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Connections:
- C3 pad 1: /ISOL_OUTPUT -> /ISOL_GND
- IC1 pad 1: /SHIFTED_x100 -> /SHIFTED_x1
- IC1 pad 7: /SHIFTED_x100 -> /SHIFTED_x10
- IC2 pad 2: Net-(IC2-Pad2) -> Net-(IC2-Pad1)
- R50 pad 2: Net-(IC2-Pad2) -> Net-(J25-Pad1)
- R52 pad 1: Net-(R52-Pad1) -> Net-(IC2-Pad1)
- R52 pad 2: Net-(IC1-Pad2) -> Net-(IC1-Pad3)
- R53 pad 1: Net-(R53-Pad1) -> Net-(IC1-Pad3)
- R53 pad 2: Net-(IC1-Pad2) -> +3.3V
- U2 pad 10: /S0 -> Net-(U2-Pad10)
- U2 pad 11: /S1 -> /S0
- U2 pad 12: /S2 -> /S1
- U2 pad 13: /S3 -> /S2
- U2 pad 14: Net-(U2-Pad14) -> /S3
- U2 pad 6: Net-(U2-Pad6) -> /SHIFTED_x1
- U2 pad 7: Net-(U2-Pad7) -> /SHIFTED_x10
- U5 pad 3: Net-(POWER_SUPPLY1-Pad2) -> /BATT
- U6 pad 16: /Dividers/OUT16 -> /Dividers/OUT13
- U6 pad 17: /Dividers/OUT15 -> /Dividers/OUT4
- U6 pad 19: /Dividers/OUT13 -> /Dividers/OUT3
- U6 pad 2: /Dividers/OUT8 -> /Dividers/OUT9
- U6 pad 20: /Dividers/OUT12 -> /Dividers/OUT15
- U6 pad 21: /Dividers/OUT11 -> /Dividers/OUT2
- U6 pad 22: /Dividers/OUT10 -> /Dividers/OUT16
- U6 pad 23: /Dividers/OUT9 -> /Dividers/OUT1
- U6 pad 3: /Dividers/OUT7 -> /Dividers/OUT8
- U6 pad 4: /Dividers/OUT6 -> /Dividers/OUT10
- U6 pad 5: /Dividers/OUT5 -> /Dividers/OUT7
- U6 pad 6: /Dividers/OUT4 -> /Dividers/OUT11
- U6 pad 7: /Dividers/OUT3 -> /Dividers/OUT6
- U6 pad 8: /Dividers/OUT2 -> /Dividers/OUT12
- U6 pad 9: /Dividers/OUT1 -> /Dividers/OUT5
Routing:
- net GND: track 0.00 -> 130.2 mm, vias 0 -> 17
- net +3.3V: track 0.00 -> 103.3 mm
- net /SHIFTED_x10: track 0.00 -> 45.0 mm, vias 0 -> 2
- net /SHIFTED_x1: track 0.00 -> 38.5 mm, vias 0 -> 2
- net /Dividers/OUT1: track 0.00 -> 33.1 mm
- net /Dividers/OUT8: track 0.00 -> 30.0 mm
- net /Dividers/OUT9: track 0.00 -> 29.5 mm, vias 0 -> 1
- net /S1: track 0.00 -> 29.1 mm
- net /S2: track 0.00 -> 28.7 mm
- net /Dividers/OUT16: track 0.00 -> 28.4 mm, vias 0 -> 1
- net /Dividers/OUT2: track 0.00 -> 28.3 mm
- net /S0: track 0.00 -> 28.2 mm
- net /S3: track 0.00 -> 26.8 mm
- net /Dividers/OUT7: track 0.00 -> 25.5 mm
- net /Dividers/OUT10: track 0.00 -> 24.5 mm, vias 0 -> 1
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- added copper zone on B.Cu, net GND
Other:
- board outline added: 71 x 46.4 mm
- net class Default: via_dia 0.8 -> 2; via_drill 0.4 -> 0.7
- board text added: "+"
- board text added: "-"
- board text added: "0xDBFB7's Psychic Probe"
- board text added: "1"
- board text added: "3V3"
- board text added: "8"
- board text added: "GND"
- board text added: "TX"
- board text added: "The Kyrt must flow"
- board text added: "the currents of current"

Commit message: Planning on renaming the firmware in STM32Cube
Parts:
- moved C5 113.5 mm to (87.2, 169.8)
- moved IC1 113.5 mm to (74.0, 161.9)
- moved IC2 113.5 mm to (83.9, 163.8)
- moved R58 113.5 mm to (72.2, 156.7)
- moved U4 113.5 mm to (90.1, 171.6)
- moved U6 113.5 mm to (96.2, 156.8)
- moved C1 113.5 mm to (88.9, 137.4)
- moved C10 113.5 mm to (84.0, 153.6)
- moved C3 113.5 mm to (68.2, 140.0)
- moved C4 113.5 mm to (93.1, 171.1)
- moved C6 113.5 mm to (87.2, 173.1)
- moved C7 113.5 mm to (85.8, 169.8)
- moved J10 113.5 mm to (123.9, 175.2)
- moved J11 113.5 mm to (123.9, 170.2)
- moved J12 113.5 mm to (123.9, 165.2)
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Other:
- net class Default: via_drill 0.7 -> 0.81
- rule pad_to_mask_clearance: 0.2 -> 0
- board text added: "16"
- board text added: "9"
