File: hardware/probe/probe.sch (KiCad schematic (older format))
At the start: 19 parts

Commit message: I think I can simplify the amplifier a bit
Parts:
- removed IC? (x3): OPAMP-DUAL, DIP08, symbol SparkFun-IC-Amplifiers:OPAMP-DUAL
- removed J?: HEADER_4, symbol w_connectors:HEADER_4
- removed OUTPUT: (no value), symbol w_connectors:HEADER_3
- removed Y?: 8MHz, HC49US, symbol SparkFun-Clocks:CRYSTALPTH-HC49US
- added IC1: TLV9062IDR, Package_SO:SOIC-8-1EP_3.9x4.9mm_P1.27mm_EP2.35x2.35mm, symbol SparkFun-IC-Amplifiers:OPAMP-DUAL
- added IC2: AZ4580, Package_SO:SOIC-8_3.9x4.9mm_P1.27mm, symbol SparkFun-IC-Amplifiers:OPAMP-DUAL
- added J18, J? (x3): ISOL_3v3, 0xDBFB7:CAP_WIRE_CONNECTION, symbol SparkFun-Connectors:CONN_01
- added J19: ISOL_GND, 0xDBFB7:CAP_WIRE_CONNECTION, symbol SparkFun-Connectors:CONN_01
- added J20: ISOL_OUTPUT, 0xDBFB7:CAP_WIRE_CONNECTION, symbol SparkFun-Connectors:CONN_01
- added R50, R?: 50k, 0603, symbol SparkFun-Resistors:10OHM-0603-1_10W-1%
- added R51: 10k, 0603, symbol SparkFun-Resistors:10OHM-0603-1_10W-1%
- added R52, R53, R? (x2): 360r, 0603, symbol SparkFun-Resistors:10OHM-0603-1_10W-1%
- added R?: 1k, 0603, symbol SparkFun-Resistors:10OHM-0603-1_10W-1%
- added Y1: 8Mhz, HC49UP, symbol SparkFun-Clocks:CRYSTAL-8MHZSMD-HC49UP
- gave numbers to parts that had none: 12
- renumbered POWER_SUPPLY to POWER_SUPPLY1
Connections:
- net labels added: SHIFTED_x100
- wire segments 59 -> 31
Other:
- note added: "Shift by 3.3/2 (rail-to-rail)\n"

Commit message: Layout complete!
Parts:
- removed POWER_SUPPLY1: (no value), 1X02, symbol SparkFun-Connectors:CONN_02
- removed R50, R?: 50k, 0603, symbol SparkFun-Resistors:10OHM-0603-1_10W-1%
- removed R51: 10k, 0603, symbol SparkFun-Resistors:10OHM-0603-1_10W-1%
- removed R?: 1k, 0603, symbol SparkFun-Resistors:10OHM-0603-1_10W-1%
- removed U3: CAT24M01W, Package_SO:SOIC-8_3.9x4.9mm_P1.27mm, symbol Memory_EEPROM:CAT24M01W
- added C10, C11, C7: 0.1uf, 0603, symbol SparkFun-Capacitors:2.2UF-0603-10V-20%
- added C6, C9: 10uf, 0603, symbol SparkFun-Capacitors:2.2UF-0603-10V-20%
- added C8: 10UF-1206-6.3V-20%, 1206, symbol SparkFun-Capacitors:10UF-1206-6.3V-20%
- added J23: BATT, 0xDBFB7:CAP_WIRE_CONNECTION, symbol SparkFun-Connectors:CONN_01
- added J24, J25: GND, 0xDBFB7:CAP_WIRE_CONNECTION, symbol SparkFun-Connectors:CONN_01
- added R50: FUSE, 1206, symbol SparkFun-Resistors:RESISTOR1206
- added R56: 1k, 0603, symbol SparkFun-Resistors:10OHM-0603-1_10W-1%
- added R57, R58, R59, R60, R61: 10k, 0603, symbol SparkFun-Resistors:10OHM-0603-1_10W-1%
- C5: value 2.2uF -> 10uf
- IC1: footprint Package_SO:SOIC-8-1EP_3.9x4.9mm_P1.27mm_EP2.35x2.35mm -> Package_SO:SOIC-8_3.9x4.9mm_P1.27mm
- R52, R53: value 360r -> 10k
- R54, R55: renamed from R?; value 360r -> 10k
- gave numbers to parts that had none: 3
Connections:
- net labels added: BATT, SHIFTED_x1, SHIFTED_x10
- net labels removed: SHIFTED_x100
- wire segments 31 -> 38
Other:
- note added: "This could be simplified a bit by adding the \ngain to the shift amps and removing the first stage, \nbut we'd need a buffer\nhere anyway because of the \nhigh impedance of the dividers."

Commit message: Feature complete, as nearly as I can tell
Parts:
- R53, R55, R58, R59: value 10k -> 20k
Changed lines of the file:
@@
 P 9200 3500
 F 0 "R53" V 9250 3600 45  0000 L CNN
-F 1 "10k" V 9150 3600 45  0000 L CNN
+F 1 "20k" V 9150 3600 45  0000 L CNN
 F 2 "0603" H 9200 3650 20  0001 C CNN
 F 3 "" H 9200 3500 60  0001 C CNN
@@
 P 9200 4750
 F 0 "R55" V 9250 4800 45  0000 L CNN
-F 1 "10k" V 9200 4800 45  0000 L CNN
+F 1 "20k" V 9200 4800 45  0000 L CNN
 F 2 "0603" H 9200 4900 20  0001 C CNN
 F 3 "" H 9200 4750 60  0001 C CNN
@@
 P 9000 4200
 F 0 "R58" H 8950 4100 45  0000 L CNN
-F 1 "10k" H 8950 4000 45  0000 L CNN
+F 1 "20k" H 8950 4000 45  0000 L CNN
 F 2 "0603" H 9000 4350 20  0001 C CNN
 F 3 "" H 9000 4200 60  0001 C CNN
@@
 P 9000 5450
 F 0 "R59" H 8950 5350 45  0000 L CNN
-F 1 "10k" H 8950 5250 45  0000 L CNN
+F 1 "20k" H 8950 5250 45  0000 L CNN
 F 2 "0603" H 9000 5600 20  0001 C CNN
 F 3 "" H 9000 5450 60  0001 C CNN
